Commit message: Add GLUON calibration and IK stack

File: sim2sim/gluon_2L6_4L3_urdf/urdf/gluon_2L6_4L3.urdf (robot description, URDF)
Before this commit: robot gluon_2L6_4L3, 8 links, 7 joints
Joints:
- joint axis_joint_1: limit lower=-3.0 upper=3.0 effort=150.0 velocity=3.0 -> lower=-2.584484342 upper=2.584484342 effort=150.0 velocity=3.0
- joint axis_joint_2: limit lower=-1.67079632679 upper=1.42920367321 effort=150.0 velocity=3.0 -> lower=-1.623319218 upper=1.651337338 effort=150.0 velocity=3.0
- joint axis_joint_3: limit lower=-3.0 upper=3.0 effort=150.0 velocity=3.0 -> lower=-2.443782617 upper=2.395065067 effort=150.0 velocity=3.0
- joint axis_joint_4: limit lower=-3.0 upper=3.0 effort=150.0 velocity=3.0 -> lower=-2.419633194 upper=2.396012955 effort=150.0 velocity=3.0
- joint axis_joint_5: limit lower=-3.0 upper=3.0 effort=150.0 velocity=3.0 -> lower=-2.421678546 upper=2.407829882 effort=150.0 velocity=3.0
- joint axis_joint_6: limit lower=-3.0 upper=3.0 effort=150.0 velocity=3.0 -> lower=-2.617993878 upper=2.617993878 effort=150.0 velocity=3.0

File: sim2sim/gluon_2L6_4L3_urdf/urdf/gluon_2L6_4L3_sim.urdf (robot description, URDF)
Before this commit: robot gluon_2L6_4L3_sim, 7 links, 6 joints
Joints:
- joint axis_joint_1: limit lower=-3.0 upper=3.0 effort=150.0 velocity=3.0 -> lower=-2.584484342 upper=2.584484342 effort=150.0 velocity=3.0
- joint axis_joint_2: limit lower=-1.67079632679 upper=1.42920367321 effort=150.0 velocity=3.0 -> lower=-1.623319218 upper=1.651337338 effort=150.0 velocity=3.0
- joint axis_joint_3: limit lower=-3.0 upper=3.0 effort=150.0 velocity=3.0 -> lower=-2.443782617 upper=2.395065067 effort=150.0 velocity=3.0
- joint axis_joint_4: limit lower=-3.0 upper=3.0 effort=150.0 velocity=3.0 -> lower=-2.419633194 upper=2.396012955 effort=150.0 velocity=3.0
- joint axis_joint_5: limit lower=-3.0 upper=3.0 effort=150.0 velocity=3.0 -> lower=-2.421678546 upper=2.407829882 effort=150.0 velocity=3.0
- joint axis_joint_6: limit lower=-3.0 upper=3.0 effort=150.0 velocity=3.0 -> lower=-2.617993878 upper=2.617993878 effort=150.0 velocity=3.0
